File: DIVA_promicro.sch (KiCad schematic (older format))
At the start: 20 parts

Commit message: Added resistor for a LED strip signal line
Parts:
- added R4: 500, Resistor_THT:R_Axial_DIN0207_L6.3mm_D2.5mm_P7.62mm_Horizontal, symbol Device:R
- ProMicro1: symbol promicro:ProMicro -> DIVA_promicro-rescue:ProMicro-promicro
Connections:
- net at ProMicro1.2 (RX): now also R4.1; no longer LED1.1 (Pin_1)
- new net: LED1.1 (Pin_1), R4.2
Changed lines of the file:
@@
 $EndDescr
 $Comp
-L promicro:ProMicro ProMicro1
+L DIVA_promicro-rescue:ProMicro-promicro ProMicro1
 U 1 1 5DC18EEE
 P 5750 2150
@@
 	4400 1200 4400 1500
 Wire Wire Line
-	4400 1500 5050 1500
+	4400 1500 4616 1500
 $Comp
 L Connector_Generic:Conn_01x02 I2C_Conn1
@@
 	1    0    0    -1
 $EndComp
+$Comp
+L Device:R R4
+U 1 1 5E4186A0
+P 4766 1500
+F 0 "R4" V 4559 1500 50  0000 C CNN
+F 1 "500" V 4650 1500 50  0000 C CNN
+F 2 "Resistor_THT:R_Axial_DIN0207_L6.3mm_D2.5mm_P7.62mm_Horizontal" V 4696 1500 50  0001 C CNN
+F 3 "~" H 4766 1500 50  0001 C CNN
+	1    4766 1500
+	0    1    1    0
+$EndComp
+Wire Wire Line
+	4916 1500 5050 1500
 $EndSCHEMATC
